File: KiCAD/Z80-8251-PPI.sch (KiCad schematic (older format))
At the start: 37 parts, among them J1 SBC8080 BUS, J2 ADDR_JP, J3 IR JP, J4 232C-CON, J5 CON-A, J6 CON-B, J7 SERIAL JP, J8 SP JP, Q1 2SC1815, U1 74LS139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

Commit message: ロジックICで割り込みコントローラ構成を検討 ドラフト版
Parts:
- removed Q1: 2SC1815, Package_TO_SOT_THT:TO-92_Inline_Wide, symbol Transistor_BJT:2SC1815
- removed R2: 100k, Resistor_THT:R_Axial_DIN0207_L6.3mm_D2.5mm_P10.16mm_Horizontal, symbol Device:R_US
- removed R3: 1k, Resistor_THT:R_Axial_DIN0207_L6.3mm_D2.5mm_P10.16mm_Horizontal, symbol Device:R_US
- removed U5: 8259, Package_DIP:DIP-28_W15.24mm_Socket, symbol Interface:8259
- added C10, C11, C12, C13: 0.1u, Capacitor_THT:C_Rect_L4.0mm_W2.5mm_P2.50mm, symbol Z80-8251-PPI-rescue:C
- added RN1, RN2, RN3: 10k, Resistor_THT:R_Array_SIP9, symbol Device:R_Network08_US
- added U5, U7: 74HC04, Package_DIP:DIP-14_W7.62mm_Socket, symbol 74xx:74HC04
- added U8: 74HC148, Package_DIP:DIP-16_W7.62mm_Socket, symbol 74xx:74LS148
- added U9: 74HC541, Package_DIP:DIP-20_W7.62mm_Socket, symbol 74xx:74LS541
- U4: footprint Housings_DIP:DIP-16_W7.62mm_Socket -> Package_DIP:DIP-16_W7.62mm_Socket
Connections:
- net labels removed: 8259-CS
- wire segments 332 -> 440
- no-connect marks 28 -> 30
Other:
- moved on the sheet: C1, C2, C3, C4, C5, C6, C7, C8, C9, J1, J2, J3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
